Commit message: RViz shows the electric grippers' fingers, opening as the gripper does
baxter.urdf (the description the teleop's kinematics, view_teleop_frames.sh and MoveIt load) had a
placeholder box per gripper and no fingers. It now carries the real electric gripper from
rethink_ee_description as {arm}_end_effector.urdf.xacro mounts it: base mesh, extended_narrow fingers
in slot 2, paddle tips, prismatic l/r finger joints. Only the fingers are grafted: the {arm}_gripper
and endpoint frames stay put, and the links have no inertials (the xacro's are 0.01 kg m^2
placeholders), so the kinematics are unchanged: TCP offset, Jacobian, mass matrix and inverse
dynamics identical to 0.0 at a random state; 85 teleop tests pass.

The sim published the finger joints as 0 (closed) always; it now publishes the measured opening on
the real joints' travel (0 to 0.0208 m). Sim, domain 43: fingertip frames 73 mm apart open, 32 mm
closed.

File: src/baxter_description/urdf/baxter.urdf (robot description, URDF)
Before this commit: robot baxter, 49 links, 48 joints
Links:
- added link l_gripper_l_finger; collision box size=0.01 0.0135 0.1127; collision box size=0.01 0.05 0.017
- added link l_gripper_l_finger_tip; collision box size=0.042 0.0065 0.037; visual mesh filename=package://rethink_ee_description/meshes/electric_gripper/fi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
- added link l_gripper_r_finger; collision box size=0.01 0.0135 0.1127; collision box size=0.01 0.05 0.017
- added link l_gripper_r_finger_tip; collision box size=0.042 0.0065 0.037; visual mesh filename=package://rethink_ee_description/meshes/electric_gripper/fi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
- added link r_gripper_l_finger; collision box size=0.01 0.0135 0.1127; collision box size=0.01 0.05 0.017
- added link r_gripper_l_finger_tip; collision cylinder length=0.037 radius=0.008; visual mesh filename=package://rethink_ee_description/meshes/electric_gripper/fi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
- added link r_gripper_r_finger; collision box size=0.01 0.0135 0.1127; collision box size=0.01 0.05 0.017
- added link r_gripper_r_finger_tip; collision cylinder length=0.037 radius=0.008; visual mesh filename=package://rethink_ee_description/meshes/electric_gripper/fi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
- link left_gripper_base: geometry visual mesh filename=package://rethink_ee_description/meshes/electric_gripper/el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
- link right_gripper_base: geometry visual mesh filename=package://rethink_ee_description/meshes/electric_gripper/el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
Joints:
- added joint l_gripper_l_finger_joint: type prismatic, parent left_gripper_base, child l_gripper_l_finger, origin xyz=0 -0.0015 0.045 rpy=0 0 0, axis 0 1 0, limit lower=0.0 upper=0.020833 effort=20.0 velocity=5.0
- added joint l_gripper_l_finger_tip_joint: type fixed, parent l_gripper_l_finger, child l_gripper_l_finger_tip, origin xyz=0.0 0.01725 0.1127 rpy=0 0 0
- added joint l_gripper_r_finger_joint: type prismatic, parent left_gripper_base, child l_gripper_r_finger, origin xyz=0 0.0015 0.045 rpy=0 0 0, axis 0 1 0, limit lower=-0.020833 upper=0.0 effort=20.0 velocity=5.0, mimic joint=l_gripper_l_finger_joint multiplier=-1.0
- added joint l_gripper_r_finger_tip_joint: type fixed, parent l_gripper_r_finger, child l_gripper_r_finger_tip, origin xyz=0.0 -0.01725 0.1127 rpy=0 0 0
- added joint r_gripper_l_finger_joint: type prismatic, parent right_gripper_base, child r_gripper_l_finger, origin xyz=0 -0.0015 0.045 rpy=0 0 0, axis 0 1 0, limit lower=0.0 upper=0.020833 effort=20.0 velocity=5.0
- added joint r_gripper_l_finger_tip_joint: type fixed, parent r_gripper_l_finger, child r_gripper_l_finger_tip, origin xyz=0.0 0.01725 0.1127 rpy=0 0 0
- added joint r_gripper_r_finger_joint: type prismatic, parent right_gripper_base, child r_gripper_r_finger, origin xyz=0 0.0015 0.045 rpy=0 0 0, axis 0 1 0, limit lower=-0.020833 upper=0.0 effort=20.0 velocity=5.0, mimic joint=r_gripper_l_finger_joint multiplier=-1.0
- added joint r_gripper_r_finger_tip_joint: type fixed, parent r_gripper_r_finger, child r_gripper_r_finger_tip, origin xyz=0.0 -0.01725 0.1127 rpy=0 0 0
